Commit message: Add documentation, code improvement/reorganization

File: src/basicjetbot_description/urdf/basicjetbot.xacro (robot description, xacro)
@@ -1,31 +1,34 @@
 <?xml version='1.0'?>
+<!-- basicjetbot // URDF MODEL DEFINITION -->
 <robot name="basicjetbot" xmlns:xacro="http://www.ros.org/wiki/xacro">
   <xacro:include filename="$(find basicjetbot_description)/urdf/basicjetbot.gazebo" />
-  <xacro:include filename="$(find basicjetbot_description)/urdf/materials.xacro" />
-  <xacro:include filename="$(find basicjetbot_description)/urdf/macros.xacro" />
-  <link name='chassis'>
-    <inertial>
-      <mass value="0.837"/>
-      <origin xyz="0.01 0 0.05" rpy="0 0 0"/>
-      <inertia
-          ixx="0.0007576" ixy="0" ixz="0"
-          iyy="0.0015486" iyz="0"
-          izz="0.0017524"
-      />
-    </inertial>
-    <collision name='chassis_collision'>
-      <origin xyz="0 0 0.05" rpy="0 0 0"/>
+  <!-- CHASSIS -->
+  <link name="chassis">
+    <visual>
+      <origin xyz="0 0 0.05"/>
+      <geometry>
+        <box size=".135 .083 .063"/>
+      </geometry>
+    </visual>
+    <collision>
+      <origin xyz="0 0 0.05"/>
       <geometry>
         <box size=".135 .083 .063"/>
       </geometry>
     </collision>
-    <visual name='chassis_visual'>
-      <origin xyz="0 0 0.05" rpy="0 0 0"/>
+    <inertial>
+      <origin xyz="0.01 0 0.05"/>
+      <mass value="0.837"/>
+      <inertia ixx="0.0007576" ixy="0" ixz="0" iyy="0.0015486" iyz="0" izz="0.0017524"/>
+    </inertial>
+    <!-- CASTER -->
+    <visual name = "caster">
+      <origin xyz="-0.0508 0 0.0117"/>
       <geometry>
-        <box size=".135 .083 .063"/>
+        <sphere radius="0.0117"/>
       </geometry>
     </visual>
-    <collision name='caster_collision'>
-      <origin xyz="-0.0508 0 0.0117" rpy="0 0 0"/>
+    <collision>
+      <origin xyz="-0.0508 0 0.0117"/>
       <geometry>
         <sphere radius="0.0117"/>
@@ -36,80 +39,60 @@
             <mu>0</mu>
             <mu2>0</mu2>
-            <slip1>1.0</slip1>
-            <slip2>1.0</slip2>
           </ode>
         </friction>
       </surface>
     </collision>
-    <visual name='caster_visual'>
-      <origin xyz="-0.0508 0 0.0117" rpy="0 0 0"/>
+  </link>
+  <!-- WHEELS -->
+  <link name="left_wheel">
+    <visual>
+      <origin rpy="0 1.5707 1.5707"/>
       <geometry>
-        <sphere radius="0.0117"/>
+        <cylinder radius="0.03" length="0.009"/>
       </geometry>
     </visual>
-  </link>
-  <link name="left_wheel">
-    <!--origin xyz="0.1 0.13 0.1" rpy="0 1.5707 1.5707"/-->
-    <collision name="collision">
-      <origin xyz="0 0 0" rpy="0 1.5707 1.5707"/>
+    <collision>
+      <origin rpy="0 1.5707 1.5707"/>
       <geometry>
         <cylinder radius="0.03" length="0.009"/>
       </geometry>
     </collision>
-    <visual name="left_wheel_visual">
-      <origin xyz="0 0 0" rpy="0 1.5707 1.5707"/>
+    <inertial>
+      <origin rpy="0 1.5707 1.5707"/>
+      <mass value="0.03"/>
+      <inertia ixx="0.00000693" ixy="0.0" ixz="0.0" iyy="0.00000693" iyz="0.0" izz="0.00001346"/>
+    </inertial>
+  </link>
+  <link name="right_wheel">
+    <visual>
+      <origin rpy="0 1.5707 1.5707"/>
       <geometry>
         <cylinder radius="0.03" length="0.009"/>
       </geometry>
     </visual>
-    <inertial>
-      <origin xyz="0 0 0" rpy="0 1.5707 1.5707"/>
-      <mass value="0.03"/>
-      <cylinder_inertia m="0.03" r="0.03" h="0.009"/>
-      <inertia
-        ixx="0.00000693" ixy="0.0" ixz="0.0"
-        iyy="0.00000693" iyz="0.0"
-        izz="0.00001346"/>
-    </inertial>
-  </link>
-  <link name="right_wheel">
-    <!--origin xyz="0.1 -0.13 0.1" rpy="0 1.5707 1.5707"/-->
-    <collision name="collision">
-      <origin xyz="0 0 0" rpy="0 1.5707 1.5707"/>
+    <collision>
+      <origin rpy="0 1.5707 1.5707"/>
       <geometry>
         <cylinder radius="0.03" length="0.009"/>
       </geometry>
     </collision>
-    <visual name="right_wheel_visual">
-      <origin xyz="0 0 0" rpy="0 1.5707 1.5707"/>
-      <geometry>
-        <cylinder radius="0.03" length="0.009"/>
-      </geometry>
-    </visual>
     <inertial>
-      <origin xyz="0 0 0" rpy="0 1.5707 1.5707"/>
+      <origin rpy="0 1.5707 1.5707"/>
       <mass value="0.03"/>
-      <cylinder_inertia m="0.03" r="0.03" h="0.009"/>
-      <inertia
-        ixx="0.00000693" ixy="0.0" ixz="0.0"
-        iyy="0.00000693" iyz="0.0"
-        izz="0.00001346"/>
+      <inertia ixx="0.00000693" ixy="0.0" ixz="0.0" iyy="0.00000693" iyz="0.0" izz="0.00001346"/>
     </inertial>
   </link>
-  <joint type="continuous" name="left_wheel_hinge">
-    <origin xyz="0.03 0.057 0.03" rpy="0 0 0"/>
+  <!-- MOTORS -->
+  <joint type="continuous" name="left_motor">
+    <origin xyz="0.03 0.057 0.03"/>
     <child link="left_wheel"/>
     <parent link="chassis"/>
-    <axis xyz="0 1 0" rpy="0 0 0"/>
-    <limit effort="100" velocity="100"/>
-    <joint_properties damping="0.0" friction="0.0"/>
+    <axis xyz="0 1 0"/>
   </joint>
-  <joint type="continuous" name="right_wheel_hinge">
-    <origin xyz="0.03 -0.057 0.03" rpy="0 0 0"/>
+  <joint type="continuous" name="right_motor">
+    <origin xyz="0.03 -0.057 0.03"/>
     <child link="right_wheel"/>
     <parent link="chassis"/>
-    <axis xyz="0 1 0" rpy="0 0 0"/>
-    <limit effort="100" velocity="100"/>
-    <joint_properties damping="0.0" friction="0.0"/>
+    <axis xyz="0 1 0"/>
   </joint>
 </robot>

File: src/emptyroom_description/urdf/emptyroom_9x9.xacro (robot description, xacro)
@@ -1,2 +1,3 @@
+<!-- basicjetbot // URDF MODEL DEFINITION -->
 <?xml version='1.0'?>
 <robot name="emptyroom_9x9" xmlns:xacro="http://www.ros.org/wiki/xacro">

Commit message: Add collision detection & world file

File: src/basicjetbot_description/urdf/basicjetbot.xacro (robot description, xacro)
@@ -11,5 +11,5 @@
       </geometry>
     </visual>
-    <collision>
+    <collision name="chassis_collision">
       <origin xyz="0 0 0.05"/>
       <geometry>

File: src/emptyroom_description/urdf/emptyroom_9x9.xacro (robot description, xacro)
@@ -1,4 +1,4 @@
-<!-- basicjetbot // URDF MODEL DEFINITION -->
 <?xml version='1.0'?>
+<!-- emptyroom_9x9 // URDF MODEL DEFINITION -->
 <robot name="emptyroom_9x9" xmlns:xacro="http://www.ros.org/wiki/xacro">
   <xacro:property name="x_dim" value="2.7432" /> <!-- 9ft = 2.7432m -->

Commit message: Add camera, new combined Gazebo interface script

File: src/basicjetbot_description/urdf/basicjetbot.xacro (robot description, xacro)
@@ -96,3 +96,26 @@
     <axis xyz="0 1 0"/>
   </joint>
+  <!-- CAMERA -->
+  <link name="camera">
+    <visual>
+      <geometry>
+        <box size="0.01 0.01 0.01"/>
+      </geometry>
+    </visual>
+    <collision>
+      <geometry>
+        <box size="0.01 0.01 0.01"/>
+      </geometry>
+    </collision>
+    <inertial>
+      <mass value="0" />
+      <inertia ixx="0" ixy="0" ixz="0" iyy="0" iyz="0" izz="0" />
+    </inertial>
+  </link>
+  <joint name="camera_joint" type="fixed">
+    <axis xyz="0 1 0" />
+    <origin xyz="0.0725 0 0.05"/>
+    <parent link="chassis"/>
+    <child link="camera"/>
+  </joint>
 </robot>
